File: hardware/stm32-field-node.kicad_pcb (KiCad board)
At the start: 2 copper layers, 45 x 35 mm, 12 parts, among them J1 USB_C_Receptacle_USB2.0_16P, J2 Conn_01x05, U2 TLV75533PDBV

Commit message: docs: label SWD header pins on silkscreen + generate fabs
Parts:
- J2 SWD: renamed from J2
Other:
- board text added: "1 VTREF"
- board text added: "2 SWDIO"
- board text added: "3 SWCLK"
- board text added: "4 NRST"
- board text added: "5 GND"
Changed lines of the file:
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@@
 		(descr "Through hole straight pin header, 1x05, 2.54mm pitch, single row")
 		(tags "Through hole pin header THT 1x05 2.54mm single row")
-		(property "Reference" "J2"
+		(property "Reference" "J2 SWD"
 			(at 0 -2.38 0)
 			(layer "F.SilkS")
@@
 			)
 			(justify left bottom)
+		)
+	)
+	(gr_text "1 VTREF\n"
+		(at 79.25 53.5 0)
+		(layer "F.SilkS")
+		(effects
+			(font
+				(size 1 1)
+				(thickness 0.15)
+			)
+			(justify left bottom)
+		)
+	)
+	(gr_text "2 SWDIO\n"
+		(at 79.25 56 0)
+		(layer "F.SilkS")
+		(effects
+			(font
+				(size 1 1)
+				(thickness 0.15)
+			)
+			(justify left bottom)
+		)
+	)
+	(gr_text "3 SWCLK\n"
+		(at 79.25 58.5 0)
+		(layer "F.SilkS")
+		(effects
+			(font
+				(size 1 1)
+				(thickness 0.15)
+			)
+			(justify left bottom)
+		)
+	)
+	(gr_text "4 NRST\n"
+		(at 79.25 61 0)
+		(layer "F.SilkS")
+		(effects
+			(font
+				(size 1 1)
+				(thickness 0.15)
+			)
+			(justify left bottom)
+		)
+	)
+	(gr_text "5 GND"
+		(at 79.25 63.75 0)
+		(layer "F.SilkS")
+		(effects
+			(font
+				(size 1 1)
+				(thickness 0.15)
+			)
+			(justify left bottom)
